File: Life_pedal/Life_pedal.kicad_pcb (KiCad board)
At the start: 4 copper layers, 65 x 70.4 mm, 89 parts, among them IC1 LM308/OP07, J1 Barrel_Jack_Switch, J10 Conn_01x01, J11 Conn_01x01, J12 Conn_01x02, J2 AudioJack3, J3 AudioJack2, J4 Conn_01x01, J5 Conn_01x01, J6 Conn_01x01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

Commit message: Final
Parts:
- moved J12 21.6 mm to (137.9, 57.4), turned to 90 degrees
- moved J4 21.6 mm to (120.8, 59.2)
- moved J8 20.0 mm to (174.4, 59.0)
- moved C1 9.25 mm to (148.4, 52.4)
- moved D1 8.51 mm to (150.7, 48.6), turned to 0 degrees
- moved C3 4.65 mm to (144.2, 55.2)
- moved C2 3.60 mm to (152.0, 52.2)
- moved J3 2.85 mm to (157.0, 51.4)
- moved J2 2.44 mm to (123.4, 51.4)
- moved R1 1.26 mm to (145.2, 49.0)
- moved R2 1.26 mm to (146.8, 49.0)
Routing:
- net Net-(J12-Pin_2): track 5.83 -> 23.3 mm
- net SIGNAL_INPUT: track 23.2 -> 8.84 mm
- net OUTPUT: track 8.55 -> 20.6 mm
- net +9V: track 184.1 -> 178.4 mm
- net Net-(D1-A): track 7.34 -> 12.5 mm
- net Net-(J12-Pin_1): track 23.8 -> 19.7 mm
- net VCC: track 57.9 -> 54.2 mm
- net GND: track 25.5 -> 24.0 mm, vias 16 -> 295
Other:
- outline, holes or cut-outs redrawn
